Commit message: modular

File: src/primeberry/description/primeberry.urdf.xacro (robot description, xacro)
@@ -1,201 +1,15 @@
 <?xml version="1.0"?>
 <robot xmlns:xacro="http://www.ros.org/wiki/xacro" name="primeberry">
-   <xacro:include filename="materials.xacro"/>
-   <xacro:property name="pi" value="3.14159265359"/>
-   <link name="world"></link>
-   <joint name="base_joint" type="fixed">
+  <xacro:include filename="materials.xacro"/>
+  <xacro:include filename="base_link.xacro"/>
+  <xacro:include filename="wheels.xacro"/>
+  <xacro:include filename="steering_mechanism.xacro"/>
+  <xacro:include filename="gazebo_control.xacro"/>
+  <xacro:property name="pi" value="3.14159265359"/>
+  <link name="world"/>
+  <joint name="base_joint" type="fixed">
     <origin xyz="1.5 1.0 0.0" rpy="0.0 0.0 0.0"/>
     <parent link="world"/>
     <child link="base_link"/>
-   </joint>
-  <!-- Link for the base of the robot -->
-  <link name="base_link">
-    <visual>
-      <geometry>
-        <box size="0.4 0.2 0.1"/> <!-- Dimensions of the base -->
-      </geometry>
-      <material name="gray"/>
-    </visual>
-    <collision>
-      <geometry>
-        <box size="0.4 0.2 0.1"/>
-      </geometry>
-    </collision>
-    <inertial>
-      <mass value="1.0"/>
-      <inertia ixx="0.01" ixy="0.0" ixz="0.0" iyy="0.01" iyz="0.0" izz="0.01"/>
-    </inertial>
-  </link>
-  <!-- Link for the back left wheel -->
-  <link name="back_left_wheel">
-    <visual>
-      <origin rpy="0.0 ${pi/2} ${pi/2}"/>
-      <geometry>
-        <cylinder length="0.05" radius="0.05"/>
-      </geometry>
-      <material name="black"/>
-    </visual>
-    <collision>
-      <origin rpy="0.0 ${pi/2} ${pi/2}"/>
-      <geometry>
-        <cylinder length="0.05" radius="0.05"/>
-      </geometry>
-    </collision>
-    <inertial>
-      <mass value="0.1"/>
-      <inertia ixx="0.001" ixy="0.0" ixz="0.0" iyy="0.001" iyz="0.0" izz="0.001"/>
-    </inertial>
-  </link>
-  <!-- Link for the back right wheel -->
-  <link name="back_right_wheel">
-    <visual>
-      <origin rpy="0.0 ${pi/2} ${pi/2}"/>
-      <geometry>
-        <cylinder length="0.05" radius="0.05"/>
-      </geometry>
-      <material name="black"/>
-    </visual>
-    <collision>
-      <origin rpy="0.0 ${pi/2} ${pi/2}"/>
-      <geometry>
-        <cylinder length="0.05" radius="0.05"/>
-      </geometry>
-    </collision>
-    <inertial>
-      <mass value="0.1"/>
-      <inertia ixx="0.001" ixy="0.0" ixz="0.0" iyy="0.001" iyz="0.0" izz="0.001"/>
-    </inertial>
-  </link>
-  <!-- Link for the front left wheel -->
-  <link name="front_left_wheel">
-    <visual>
-      <origin rpy="0.0 ${pi/2} ${pi/2}"/>
-      <geometry>
-        <cylinder length="0.05" radius="0.05"/>
-      </geometry>
-      <material name="black"/>
-    </visual>
-    <collision>
-      <origin rpy="0.0 ${pi/2} ${pi/2}"/>
-      <geometry>
-        <cylinder length="0.05" radius="0.05"/>
-      </geometry>
-    </collision>
-    <inertial>
-      <mass value="0.1"/>
-      <inertia ixx="0.001" ixy="0.0" ixz="0.0" iyy="0.001" iyz="0.0" izz="0.001"/>
-    </inertial>
-  </link>
-  <!-- Link for the front right wheel -->
-  <link name="front_right_wheel">
-    <visual>
-      <origin rpy="0.0 ${pi/2} ${pi/2}"/>
-      <geometry>
-        <cylinder length="0.05" radius="0.05"/>
-      </geometry>
-      <material name="black"/>
-    </visual>
-    <collision>
-      <origin rpy="0.0 ${pi/2} ${pi/2}"/>
-      <geometry>
-        <cylinder length="0.05" radius="0.05"/>
-      </geometry>
-    </collision>
-    <inertial>
-      <mass value="0.1"/>
-      <inertia ixx="0.001" ixy="0.0" ixz="0.0" iyy="0.001" iyz="0.0" izz="0.001"/>
-    </inertial>
-  </link>
-  <!-- Joint for the back left wheel -->
-  <joint name="back_left_wheel_joint" type="continuous">
-    <parent link="base_link"/>
-    <child link="back_left_wheel"/>
-    <origin xyz="-0.2 -0.125 0"/>
-    <axis xyz="0 1 0"/>
-  </joint>
-  <!-- Joint for the back right wheel -->
-  <joint name="back_right_wheel_joint" type="continuous">
-    <parent link="base_link"/>
-    <child link="back_right_wheel"/>
-    <origin xyz="-0.2 0.125 0"/>
-    <axis xyz="0 1 0"/>
-  </joint>
-  <!-- Joint for the front left wheel -->
-  <!-- <joint name="front_left_wheel_joint" type="continuous">
-    <parent link="base_link"/>
-    <child link="front_left_wheel"/>
-    <origin xyz="0.2 -0.1 0"/>
-    <axis xyz="0 1 0"/>
-  </joint> -->
-  <!-- Joint for the front right wheel -->
-  <!-- <joint name="front_right_wheel_joint" type="continuous">
-    <parent link="base_link"/>
-    <child link="front_right_wheel"/>
-    <origin xyz="0.2 0.1 0"/>
-    <axis xyz="0 1 0"/>
-  </joint> -->
-  <!-- Link for the sphere -->
-  <link name="steering_sphere">
-    <visual>
-      <geometry>
-        <sphere radius="0.025"/>
-      </geometry>
-      <material name="blue"/>
-    </visual>
-    <collision>
-      <geometry>
-        <sphere radius="0.025"/>
-      </geometry>
-    </collision>
-    <inertial>
-      <mass value="0.05"/>
-      <inertia ixx="0.0001" ixy="0.0" ixz="0.0" iyy="0.0001" iyz="0.0" izz="0.0001"/>
-    </inertial>
-  </link>
-  <!-- Joint connecting the sphere to the base link -->
-  <joint name="sphere_to_base_joint" type="fixed">
-    <parent link="base_link"/>
-    <child link="steering_sphere"/>
-    <origin xyz="0.225 0 0"/>
-  </joint>
-  <!-- Joint connecting the sphere to the steering mechanism -->
-  <joint name="sphere_to_steering_joint" type="revolute">
-    <parent link="steering_sphere"/>
-    <child link="front_wheel_steering_link"/>
-    <origin xyz="0.075 0 0"/> <!-- Position the sphere below the steering mechanism -->
-    <axis xyz="0 0 1"/> <!-- Define the axis of rotation -->
-    <limit lower="-0.75" upper="0.75" effort="1.0" velocity="1.0"/> <!-- Define the limits, effort, and velocity -->
-  </joint>
-  <!-- Link for the steering mechanism -->
-  <link name="front_wheel_steering_link">
-    <visual>
-      <geometry>
-        <box size="0.1 0.2 0.05"/>
-      </geometry>
-      <material name="gray"/>
-    </visual>
-    <collision>
-      <geometry>
-        <box size="0.1 0.2 0.05"/>
-      </geometry>
-    </collision>
-    <inertial>
-      <mass value="0.2"/>
-      <inertia ixx="0.002" ixy="0.0" ixz="0.0" iyy="0.002" iyz="0.0" izz="0.002"/>
-    </inertial>
-  </link>
-  <!-- Joint for the front left wheel attached to the steering mechanism -->
-  <joint name="front_left_wheel_steering_joint" type="continuous">
-    <parent link="front_wheel_steering_link"/>
-    <child link="front_left_wheel"/>
-    <origin xyz="0 -0.125 0"/>
-    <axis xyz="0 1 0"/>
-  </joint>
-  <!-- Joint for the front right wheel attached to the steering mechanism -->
-  <joint name="front_right_wheel_steering_joint" type="continuous">
-    <parent link="front_wheel_steering_link"/>
-    <child link="front_right_wheel"/>
-    <origin xyz="0 0.125 0"/>
-    <axis xyz="0 1 0"/>
   </joint>
 </robot>
