Commit message: trying primeberry

File: src/primeberry/description/gazebo_control.xacro (robot description, xacro)
@@ -1,7 +1,43 @@
 <?xml version="1.0"?>
-<robot xmlns:xacro="http://www.ros.org/wiki/xacro" name="primeberry">
-    <gazebo>
-        <plugin name="ack_drive" filename="libgazebo_ros_control.so">
-        </plugin>
-    </gazebo>
+<robot xmlns:xacro="http://www.ros.org/wiki/xacro">
+	<gazebo>
+		<plugin name="gazebo_ackermann_drive" filename="libgazebo_ros_ackermann_drive.so">
+  <ros>
+    <namespace>ack</namespace>
+    <remapping>cmd_vel:=cmd_vel</remapping>
+    <remapping>odom:=odom</remapping>
+    <remapping>distance:=distance</remapping>
+  </ros>
+  <update_rate>100.0</update_rate>
+  <!-- wheels -->
+  <front_left_joint>front_left_wheel_joint</front_left_joint>
+  <front_right_joint>front_right_wheel_joint</front_right_joint>
+  <rear_left_joint>back_left_wheel_joint</rear_left_joint>
+  <rear_right_joint>back_left_wheel_joint</rear_right_joint>
+  <left_steering_joint>front_left_wheel_steering_joint</left_steering_joint>
+  <right_steering_joint>front_right_wheel_steering_joint</right_steering_joint>
+  <steering_wheel_joint>sphere_to_base_joint</steering_wheel_joint>
+  <!-- Max absolute steer angle for tyre in radians-->
+  <!-- Any cmd_vel angular z greater than this would be capped -->
+  <max_steer>0.6458</max_steer>
+  <!-- Max absolute steering angle of steering wheel -->
+  <max_steering_angle>7.85</max_steering_angle>
+  <!-- Max absolute linear speed in m/s -->
+  <max_speed>20</max_speed>
+  <!-- PID tuning -->
+  <left_steering_pid_gain>1500 0 1</left_steering_pid_gain>
+  <left_steering_i_range>0 0</left_steering_i_range>
+  <right_steering_pid_gain>1500 0 1</right_steering_pid_gain>
+  <right_steering_i_range>0 0</right_steering_i_range>
+  <linear_velocity_pid_gain>1000 0 1</linear_velocity_pid_gain>
+  <linear_velocity_i_range>0 0</linear_velocity_i_range>
+  <!-- output -->
+  <publish_odom>true</publish_odom>
+  <publish_odom_tf>true</publish_odom_tf>
+  <publish_wheel_tf>true</publish_wheel_tf>
+  <publish_distance>true</publish_distance>
+  <odometry_frame>odom</odometry_frame>
+  <robot_base_frame>chassis</robot_base_frame>
+</plugin>
+	</gazebo>
 </robot>

File: src/primeberry/description/steering_mechanism.xacro (robot description, xacro)
@@ -30,8 +30,10 @@
     </gazebo>
     <!-- Joint connecting the sphere to the base link -->
-    <joint name="sphere_to_base_joint" type="fixed">
+    <joint name="sphere_to_base_joint" type="revolute">
       <parent link="base_link"/>
       <child link="steering_sphere"/>
       <origin xyz="0.225 0 0"/>
+      <axis xyz="0 1 0"/>
+      <limit lower="-0.75" upper="0.75" effort="1.0" velocity="1.0"/>
     </joint>
     <!-- Joint connecting the sphere to the steering mechanism -->
@@ -40,5 +42,5 @@
       <child link="front_wheel_steering_link"/>
       <origin xyz="0.075 0 0"/> <!-- Position the sphere below the steering mechanism -->
-      <axis xyz="0 0 1"/> <!-- Define the axis of rotation -->
+      <axis xyz="0 1 0"/> <!-- Define the axis of rotation -->
       <limit lower="-0.75" upper="0.75" effort="1.0" velocity="1.0"/> <!-- Define the limits, effort, and velocity -->
     </joint>
@@ -66,15 +68,29 @@
     </gazebo>
     <!-- Joints for the front wheels attached to the steering mechanism -->
-    <joint name="front_left_wheel_steering_joint" type="continuous">
+    <!-- <joint name="front_left_wheel_joint" type="continuous">
       <parent link="front_wheel_steering_link"/>
       <child link="front_left_wheel"/>
       <origin xyz="0 -0.125 0"/>
       <axis xyz="0 1 0"/>
+    </joint> -->
+     <joint name="front_left_wheel_steering_joint" type="revolute">
+      <parent link="front_wheel_steering_link"/>
+      <child link="front_left_wheel"/>
+      <origin xyz="0 -0.125 0"/>
+      <axis xyz="0 0 1"/>
+      <limit lower="-0.75" upper="0.75" effort="1.0" velocity="1.0"/>
     </joint>
-    <joint name="front_right_wheel_steering_joint" type="continuous">
+    <!-- <joint name="front_right_wheel_joint" type="continuous">
       <parent link="front_wheel_steering_link"/>
       <child link="front_right_wheel"/>
       <origin xyz="0 0.125 0"/>
       <axis xyz="0 1 0"/>
+    </joint> -->
+    <joint name="front_right_wheel_steering_joint" type="revolute">
+      <parent link="front_wheel_steering_link"/>
+      <child link="front_right_wheel"/>
+      <origin xyz="0 0.125 0"/>
+      <axis xyz="0 0 1"/>
+      <limit lower="-0.75" upper="0.75" effort="1.0" velocity="1.0"/>
     </joint>
 </robot>

File: src/primeberry_one/description/gazebo_control.xacro (robot description, xacro)
@@ -36,5 +36,5 @@
   <publish_wheel_tf>true</publish_wheel_tf>
   <publish_distance>true</publish_distance>
-  <odometry_frame>odom_demo</odometry_frame>
+  <odometry_frame>odom</odometry_frame>
   <robot_base_frame>chassis</robot_base_frame>
 </plugin>
