Commit message: steering axis fix

File: src/primeberry/description/steering_mechanism.xacro (robot description, xacro)
@@ -34,5 +34,5 @@
       <child link="steering_sphere"/>
       <origin xyz="0.225 0 0"/>
-      <axis xyz="0 1 0"/>
+      <axis xyz="1 0 0"/>
       <limit lower="-0.75" upper="0.75" effort="1.0" velocity="1.0"/>
     </joint>
@@ -42,6 +42,7 @@
       <child link="front_wheel_steering_link"/>
       <origin xyz="0.075 0 0"/> <!-- Position the sphere below the steering mechanism -->
-      <axis xyz="0 1 0"/> <!-- Define the axis of rotation -->
+      <axis xyz="1 0 0"/> <!-- Define the axis of rotation -->
       <limit lower="-0.75" upper="0.75" effort="1.0" velocity="1.0"/> <!-- Define the limits, effort, and velocity -->
+      <dynamics damping="0.0" friction="0.0"/> <!-- Set dynamics to frictionless -->
     </joint>
     <!-- Link for the steering mechanism -->
@@ -68,10 +69,10 @@
     </gazebo>
     <!-- Joints for the front wheels attached to the steering mechanism -->
-    <!-- <joint name="front_left_wheel_joint" type="continuous">
+    <joint name="front_left_wheel_joint" type="continuous">
       <parent link="front_wheel_steering_link"/>
       <child link="front_left_wheel"/>
       <origin xyz="0 -0.125 0"/>
       <axis xyz="0 1 0"/>
-    </joint> -->
+    </joint>
      <joint name="front_left_wheel_steering_joint" type="revolute">
       <parent link="front_wheel_steering_link"/>
@@ -81,10 +82,10 @@
       <limit lower="-0.75" upper="0.75" effort="1.0" velocity="1.0"/>
     </joint>
-    <!-- <joint name="front_right_wheel_joint" type="continuous">
+    <joint name="front_right_wheel_joint" type="continuous">
       <parent link="front_wheel_steering_link"/>
       <child link="front_right_wheel"/>
       <origin xyz="0 0.125 0"/>
       <axis xyz="0 1 0"/>
-    </joint> -->
+    </joint>
     <joint name="front_right_wheel_steering_joint" type="revolute">
       <parent link="front_wheel_steering_link"/>
