Commit message: removed steering mechanism

File: src/primeberry_one/description/gazebo_control.xacro (robot description, xacro)
@@ -2,8 +2,41 @@
 <robot xmlns:xacro="http://www.ros.org/wiki/xacro">
 	<gazebo>
-		<plugin name="gazebo_ros_control" filename="libgazebo_ros_control.so">
-		  <robotNamespace>/ack</robotNamespace>
-			<legacyModeNS>true</legacyModeNS>
-		</plugin>
+		<plugin name="gazebo_ackermann_drive" filename="libgazebo_ros_ackermann_drive.so">
+  <ros>
+    <namespace>demo</namespace>
+    <remapping>cmd_vel:=cmd_demo</remapping>
+    <remapping>odom:=odom_demo</remapping>
+    <remapping>distance:=distance_demo</remapping>
+  </ros>
+  <update_rate>100.0</update_rate>
+  <!-- wheels -->
+  <front_left_joint>front_left_wheel_rotate</front_left_joint>
+  <front_right_joint>front_right_wheel_rotate</front_right_joint>
+  <rear_left_joint>left_wheel_rear_rotate</rear_left_joint>
+  <rear_right_joint>right_wheel_rear_rotate</rear_right_joint>
+  <left_steering_joint>front_left_wheel_hinge</left_steering_joint>
+  <right_steering_joint>front_right_wheel_hinge</right_steering_joint>
+  <!-- Max absolute steer angle for tyre in radians-->
+  <!-- Any cmd_vel angular z greater than this would be capped -->
+  <max_steer>0.6458</max_steer>
+  <!-- Max absolute steering angle of steering wheel -->
+  <max_steering_angle>7.85</max_steering_angle>
+  <!-- Max absolute linear speed in m/s -->
+  <max_speed>20</max_speed>
+  <!-- PID tuning -->
+  <left_steering_pid_gain>1500 0 1</left_steering_pid_gain>
+  <left_steering_i_range>0 0</left_steering_i_range>
+  <right_steering_pid_gain>1500 0 1</right_steering_pid_gain>
+  <right_steering_i_range>0 0</right_steering_i_range>
+  <linear_velocity_pid_gain>1000 0 1</linear_velocity_pid_gain>
+  <linear_velocity_i_range>0 0</linear_velocity_i_range>
+  <!-- output -->
+  <publish_odom>true</publish_odom>
+  <publish_odom_tf>true</publish_odom_tf>
+  <publish_wheel_tf>true</publish_wheel_tf>
+  <publish_distance>true</publish_distance>
+  <odometry_frame>odom_demo</odometry_frame>
+  <robot_base_frame>chassis</robot_base_frame>
+</plugin>
 	</gazebo>
 </robot>

File: src/primeberry_one/description/primeberry_one.urdf.xacro (robot description, xacro)
@@ -45,5 +45,5 @@
 	<!-- Chassis END -->
   <!-- Right Wheel - Start -->
-	<link name="right_wheel">
+	<link name="front_right_wheel">
 		<collision>
 		  <origin xyz="0 0 0" rpy="0 1.5708 1.5708" />
@@ -66,5 +66,5 @@
 	  </inertial>
 	</link>
-  <gazebo reference="right_wheel">
+  <gazebo reference="front_right_wheel">
     <mu1 value="2.0"/>
     <mu2 value="2.0"/>
@@ -74,5 +74,5 @@
     <material>Gazebo/Blue</material>
   </gazebo>
-	<link name="right_wheel_assembly">
+	<link name="front_right_wheel_assembly">
 		<collision>
 		  <origin xyz="0 0 0" rpy="0 1.5708 1.5708" />
@@ -95,5 +95,5 @@
 	  </inertial>
 	</link>
-  <gazebo reference="right_wheel_assembly">
+  <gazebo reference="front_right_wheel_assembly">
     <mu1 value="2.0"/>
     <mu2 value="2.0"/>
@@ -103,7 +103,7 @@
     <material>Gazebo/White</material>
   </gazebo>
-  <joint name="right_wheel_hinge" type="revolute">
+  <joint name="front_right_wheel_hinge" type="revolute">
     <parent link="chassis"/>
-    <child link="right_wheel_assembly"/>
+    <child link="front_right_wheel_assembly"/>
     <origin xyz="0.4 0.125 0.3" rpy="0 0 0" />
     <axis xyz="0 0 1" rpy="0 0 0" />
@@ -111,7 +111,7 @@
     <dynamics damping="0.0" friction="0.0"/>
   </joint>
-  <joint name="right_wheel_rotate" type="continuous">
-    <parent link="right_wheel_assembly"/>
-    <child link="right_wheel"/>
+  <joint name="front_right_wheel_rotate" type="continuous">
+    <parent link="front_right_wheel_assembly"/>
+    <child link="front_right_wheel"/>
     <origin xyz="0.0 0.025 0.0" rpy="0 0 0" />
     <axis xyz="0 1 0" rpy="0 0 0" />
@@ -119,7 +119,7 @@
     <dynamics damping="0.0" friction="0.0"/>
   </joint>
-  <transmission name="trans_right_wheel_hing">
+  <transmission name="trans_front_right_wheel_hing">
     <type>transmission_interface/SimpleTransmission</type>
-    <joint name="right_wheel_hinge">
+    <joint name="front_right_wheel_hinge">
       <hardwareInterface>EffortJointInterface</hardwareInterface>
     </joint>
@@ -129,10 +129,10 @@
     </actuator>
   </transmission>
-  <transmission name="trans_right_wheel_rotate">
+  <transmission name="trans_front_right_wheel_rotate">
     <type>transmission_interface/SimpleTransmission</type>
-    <joint name="right_wheel_rotate">
+    <joint name="front_right_wheel_rotate">
       <hardwareInterface>EffortJointInterface</hardwareInterface>
     </joint>
-    <actuator name="motor_right_wheel_rotate">
+    <actuator name="motor_front_right_wheel_rotate">
       <hardwareInterface>EffortJointInterface</hardwareInterface>
       <mechanicalReduction>1</mechanicalReduction>
@@ -141,5 +141,5 @@
   <!-- Right Wheel - End -->
   <!-- Left Wheel - Start  -->
-	<link name="left_wheel">
+	<link name="front_left_wheel">
 		<collision>
 		  <origin xyz="0 0 0" rpy="0 1.5708 1.5708" />
@@ -162,5 +162,5 @@
 	  </inertial>
 	</link>
-  <gazebo reference="left_wheel">
+  <gazebo reference="front_left_wheel">
     <mu1 value="2.0"/>
     <mu2 value="2.0"/>
@@ -170,5 +170,5 @@
     <material>Gazebo/Blue</material>
   </gazebo>
-	<link name="left_wheel_assembly">
+	<link name="front_left_wheel_assembly">
 		<collision>
 		  <origin xyz="0 0 0" rpy="0 1.5708 1.5708" />
@@ -191,5 +191,5 @@
 	  </inertial>
 	</link>
-  <gazebo reference="left_wheel_assembly">
+  <gazebo reference="front_left_wheel_assembly">
     <mu1 value="2.0"/>
     <mu2 value="2.0"/>
@@ -199,7 +199,7 @@
     <material>Gazebo/White</material>
   </gazebo>
-  <joint name="left_wheel_hinge" type="revolute">
+  <joint name="front_left_wheel_hinge" type="revolute">
     <parent link="chassis"/>
-    <child link="left_wheel_assembly"/>
+    <child link="front_left_wheel_assembly"/>
     <origin xyz="0.4 -0.125 0.3" rpy="0 0 0" />
     <axis xyz="0 0 1" rpy="0 0 0" />
@@ -207,7 +207,7 @@
     <dynamics damping="0.0" friction="0.0"/>
   </joint>
-  <joint name="left_wheel_rotate" type="continuous">
-    <parent link="left_wheel_assembly"/>
-    <child link="left_wheel"/>
+  <joint name="front_left_wheel_rotate" type="continuous">
+    <parent link="front_left_wheel_assembly"/>
+    <child link="front_left_wheel"/>
     <origin xyz="0.0 -0.025 0.0" rpy="0 0 0" />
     <axis xyz="0 1 0" rpy="0 0 0" />
@@ -217,5 +217,5 @@
   <transmission name="tran2">
     <type>transmission_interface/SimpleTransmission</type>
-    <joint name="left_wheel_hinge">
+    <joint name="front_left_wheel_hinge">
       <hardwareInterface>EffortJointInterface</hardwareInterface>
     </joint>
@@ -225,10 +225,10 @@
     </actuator>
   </transmission>
-  <transmission name="trans_left_wheel_rotate">
+  <transmission name="trans_front_left_wheel_rotate">
     <type>transmission_interface/SimpleTransmission</type>
-    <joint name="left_wheel_rotate">
+    <joint name="front_left_wheel_rotate">
       <hardwareInterface>EffortJointInterface</hardwareInterface>
     </joint>
-    <actuator name="motor_left_wheel_rotate">
+    <actuator name="motor_front_left_wheel_rotate">
       <hardwareInterface>EffortJointInterface</hardwareInterface>
       <mechanicalReduction>1</mechanicalReduction>
