Commit message: don't know

File: src/primeberry_one/description/primeberry_one.urdf.xacro (robot description, xacro)
@@ -19,5 +19,4 @@
     </collision>
     <visual>
-      <!-- <origin xyz="0 0 0.3" rpy="0 0 0"/>  -->
       <geometry>
          <box size="1 0.2 0.1"/>
@@ -27,5 +26,4 @@
     <inertial>
       <mass value="1"/>
-      <!-- <origin xyz="0 0 0.3" rpy="0 0 0"/>  -->
       <inertia ixx="0.4" ixy="0.1" ixz="0.1" iyy="0.4" iyz="0.1" izz="0.2"/>
     </inertial>
@@ -87,5 +85,5 @@
 			<cylinder length="0.001" radius="0.04"/>
 		  </geometry>
-		  <material name="white"/>
+		  <material name="black"/>
 		</visual>
 		<inertial>
@@ -102,5 +100,5 @@
     <kd  value="1.0" />
     <fdir1 value="0 1 0"/>
-    <material>Gazebo/White</material>
+    <material>Gazebo/Black</material>
   </gazebo>
   <joint name="front_right_wheel_hinge" type="revolute">
@@ -169,5 +167,5 @@
     <kd  value="1.0" />
     <fdir1 value="0 1 0"/>
-    <material>Gazebo/Blue</material>
+    <material>Gazebo/Black</material>
   </gazebo>
 	<link name="front_left_wheel_assembly">
@@ -183,5 +181,5 @@
 			<cylinder length="0.001" radius="0.04"/>
 		  </geometry>
-		  <material name="white"/>
+		  <material name="black"/>
 		</visual>
 		<inertial>
@@ -198,5 +196,5 @@
     <kd  value="1.0" />
     <fdir1 value="0 1 0"/>
-    <material>Gazebo/White</material>
+    <material>Gazebo/Black</material>
   </gazebo>
   <joint name="front_left_wheel_hinge" type="revolute">
@@ -273,5 +271,5 @@
     <kd  value="1.0" />
     <fdir1 value="0 1 0"/>
-    <material>Gazebo/Blue</material>
+    <material>Gazebo/Black</material>
   </gazebo>
   <!-- Right Rear Wheel End -->
@@ -315,3 +313,9 @@
   </gazebo>
   <!-- Left Rear Wheel End -->
+	<gazebo>
+		<plugin name="gazebo_ros_control" filename="libgazebo_ros_control.so">
+		  <robotNamespace>/ack</robotNamespace>
+			<legacyModeNS>true</legacyModeNS>
+		</plugin>
+	</gazebo>
 </robot>

Commit message: please work

File: src/primeberry_one/description/primeberry_one.urdf.xacro (robot description, xacro)
@@ -105,5 +105,5 @@
     <parent link="chassis"/>
     <child link="front_right_wheel_assembly"/>
-    <origin xyz="0.4 0.125 0.0" rpy="0 0 0" />
+    <origin xyz="0.4 0.1005 0.0" rpy="0 0 0" />
     <axis xyz="0 0 1" rpy="0 0 0" />
     <limit effort="100" velocity="1" lower="-1" upper="1"/>
@@ -201,5 +201,5 @@
     <parent link="chassis"/>
     <child link="front_left_wheel_assembly"/>
-    <origin xyz="0.4 -0.125 0.0" rpy="0 0 0" />
+    <origin xyz="0.4 -0.1005 0.0" rpy="0 0 0" />
     <axis xyz="0 0 1" rpy="0 0 0" />
     <limit effort="100" velocity="1" lower="-1" upper="1"/>
@@ -260,5 +260,5 @@
     <parent link="chassis"/>
     <child link="right_wheel_rear"/>
-    <origin xyz="-0.4 0.15 0.0" rpy="0 0 0" />
+    <origin xyz="-0.4 0.125 0.0" rpy="0 0 0" />
     <axis xyz="0 1 0" rpy="0 0 0" />
     <limit effort="0" velocity="0"/>
@@ -299,5 +299,5 @@
     <parent link="chassis"/>
     <child link="left_wheel_rear"/>
-    <origin xyz="-0.4 -0.15 0.0" rpy="0 0 0" />
+    <origin xyz="-0.4 -0.125 0.0" rpy="0 0 0" />
     <axis xyz="0 1 0" rpy="0 0 0" />
     <limit effort="0" velocity="0"/>
@@ -313,9 +313,3 @@
   </gazebo>
   <!-- Left Rear Wheel End -->
-	<gazebo>
-		<plugin name="gazebo_ros_control" filename="libgazebo_ros_control.so">
-		  <robotNamespace>/ack</robotNamespace>
-			<legacyModeNS>true</legacyModeNS>
-		</plugin>
-	</gazebo>
 </robot>
