Commit message: build files

File: install/primeberry_one/share/primeberry_one/description/primeberry_one.urdf.xacro (robot description, xacro)
@@ -1,15 +1,11 @@
 <?xml version="1.0"?>
-<robot name="ackermann_1" xmlns:xacro="http://www.ros.org/wiki/xacro">
-	<!-- Base link -->
-  <link name="base_link">
-    <visual>
-      <geometry>
-        <box size="0.01 0.01 0.01"/>
-      </geometry>
-    </visual>
+<robot name="primeberry_one" xmlns:xacro="http://www.ros.org/wiki/xacro">
+	<!-- World link -->
+  <link name="world">
   </link>
 	<!-- Chassis START-->
 	<joint name="base_joint" type="fixed">
-    <parent link="base_link"/>
+        <origin xyz="1.5 1.0 0.0"/>
+    <parent link="world"/>
     <child link="chassis"/>
   </joint>

Commit message: build files

File: install/primeberry_one/share/primeberry_one/description/primeberry_one.urdf.xacro (robot description, xacro)
@@ -19,5 +19,4 @@
     </collision>
     <visual>
-      <!-- <origin xyz="0 0 0.3" rpy="0 0 0"/>  -->
       <geometry>
          <box size="1 0.2 0.1"/>
@@ -27,5 +26,4 @@
     <inertial>
       <mass value="1"/>
-      <!-- <origin xyz="0 0 0.3" rpy="0 0 0"/>  -->
       <inertia ixx="0.4" ixy="0.1" ixz="0.1" iyy="0.4" iyz="0.1" izz="0.2"/>
     </inertial>
@@ -87,5 +85,5 @@
 			<cylinder length="0.001" radius="0.04"/>
 		  </geometry>
-		  <material name="white"/>
+		  <material name="black"/>
 		</visual>
 		<inertial>
@@ -102,10 +100,10 @@
     <kd  value="1.0" />
     <fdir1 value="0 1 0"/>
-    <material>Gazebo/White</material>
+    <material>Gazebo/Black</material>
   </gazebo>
   <joint name="front_right_wheel_hinge" type="revolute">
     <parent link="chassis"/>
     <child link="front_right_wheel_assembly"/>
-    <origin xyz="0.4 0.125 0.0" rpy="0 0 0" />
+    <origin xyz="0.4 0.1005 0.0" rpy="0 0 0" />
     <axis xyz="0 0 1" rpy="0 0 0" />
     <limit effort="100" velocity="1" lower="-1" upper="1"/>
@@ -169,5 +167,5 @@
     <kd  value="1.0" />
     <fdir1 value="0 1 0"/>
-    <material>Gazebo/Blue</material>
+    <material>Gazebo/Black</material>
   </gazebo>
 	<link name="front_left_wheel_assembly">
@@ -183,5 +181,5 @@
 			<cylinder length="0.001" radius="0.04"/>
 		  </geometry>
-		  <material name="white"/>
+		  <material name="black"/>
 		</visual>
 		<inertial>
@@ -198,10 +196,10 @@
     <kd  value="1.0" />
     <fdir1 value="0 1 0"/>
-    <material>Gazebo/White</material>
+    <material>Gazebo/Black</material>
   </gazebo>
   <joint name="front_left_wheel_hinge" type="revolute">
     <parent link="chassis"/>
     <child link="front_left_wheel_assembly"/>
-    <origin xyz="0.4 -0.125 0.0" rpy="0 0 0" />
+    <origin xyz="0.4 -0.1005 0.0" rpy="0 0 0" />
     <axis xyz="0 0 1" rpy="0 0 0" />
     <limit effort="100" velocity="1" lower="-1" upper="1"/>
@@ -262,5 +260,5 @@
     <parent link="chassis"/>
     <child link="right_wheel_rear"/>
-    <origin xyz="-0.4 0.15 0.0" rpy="0 0 0" />
+    <origin xyz="-0.4 0.125 0.0" rpy="0 0 0" />
     <axis xyz="0 1 0" rpy="0 0 0" />
     <limit effort="0" velocity="0"/>
@@ -273,5 +271,5 @@
     <kd  value="1.0" />
     <fdir1 value="0 1 0"/>
-    <material>Gazebo/Blue</material>
+    <material>Gazebo/Black</material>
   </gazebo>
   <!-- Right Rear Wheel End -->
@@ -301,5 +299,5 @@
     <parent link="chassis"/>
     <child link="left_wheel_rear"/>
-    <origin xyz="-0.4 -0.15 0.0" rpy="0 0 0" />
+    <origin xyz="-0.4 -0.125 0.0" rpy="0 0 0" />
     <axis xyz="0 1 0" rpy="0 0 0" />
     <limit effort="0" velocity="0"/>
