Commit message: slammming it

File: src/primeberry_two/description/em_3905.urdf.xacro (robot description, xacro)
@@ -305,4 +305,11 @@
                  lr_reflect="${lr_reflect}"/>
   </xacro:macro>
+  <joint name="base_footprint_joint" type="fixed">
+      <origin xyz="0.0 0.0 0.0" rpy="0 0 0"/>
+    <parent link="base_link"/>
+    <child link="base_footprint"/>
+  </joint>
+  <link name="base_footprint">
+  </link>
   <!-- base_link must have geometry so that its axes can be displayed in
        rviz. -->

Commit message: trying nav2

File: src/primeberry_two/description/em_3905.urdf.xacro (robot description, xacro)
@@ -36,5 +36,5 @@
   <xacro:property name="chassis_length" value="0.258"/>
   <xacro:property name="chassis_width" value="0.168"/>
-  <xacro:property name="chassis_height" value="0.05"/>
+  <xacro:property name="chassis_height" value="0.1"/>
   <xacro:property name="chassis_mass" value="2.788"/>
   <!-- battery_dist is the distance between the inner edges of the
@@ -59,5 +59,5 @@
   <xacro:property name="tire_width" value="0.0689"/>
   <xacro:property name="hex_hub_depth" value="0.01445"/>
-  <xacro:property name="wheel_mass" value="0.29"/>
+  <xacro:property name="wheel_mass" value="0.59"/>
   <!-- hex_hub_dist is the distance between left and right hex hubs when
        the shock absorbers are fully extended. axle_length is the distance
@@ -370,5 +370,5 @@
       <ros>
         <namespace>/</namespace>
-        <remapping>cmd_vel:=cmd_vel</remapping>
+        <remapping>cmd_vel:=cmd_vel_nav</remapping>
         <remapping>odom:=odom</remapping>
         <remapping>distance:=distance</remapping>

File: src/primeberry_two/description/lidar.xacro (robot description, xacro)
@@ -13,5 +13,5 @@
         <parent link="chassis"/>
         <child link="laser_frame"/>
-        <origin xyz="0.1 0 0.045" rpy="0 0 0"/>
+        <origin xyz="0.1 0 0.07" rpy="0 0 0"/>
     </joint>
     <link name="laser_frame">
